File: apollobvm_pcb.sch (EAGLE design)
At the start: 21 parts, among them IC1 ATMEGA328-20P, IC2 ATMEGA328-20P, X1 22-23-2031, X2 22-23-2031, X3 22-23-2021, X4 22-23-2051, X5 22-23-2021

Commit message: Finished initial board
Parts:
- removed SV1: (no value), con-lstb:MA03-1
- removed X3, X5: 22-23-2021, con-molex:22-23-2021
- removed X4: 22-23-2051, con-molex:22-23-2051
- added BUTTON, PWR_IN: 22-23-2021, con-molex:22-23-2021
- added DISPLAY, MST_PRGM, SLV_PRGM: (no value), con-lstb:MA03-1
- added ENC: 22-23-2051, con-molex:22-23-2051
- added MST_BOOT, SLV_BOOT: (no value), con-lstb:MA04-1
- Q1, Q2: device special:XTAL/S -> apollobvm_pcb:XTAL/S
- renumbered IC1 to MASTER, IC2 to SLAVE, X1 to SER_1, X2 to SER_2
Connections:
- new net N$15: SLAVE.(PCI3/MOSI/OC2A)PB3, SLV_BOOT.1
- new net N$16: SLAVE.(PCI4/MISO)PB4, SLV_BOOT.2
- new net N$17: SLAVE.(PCI5/SCK)PB5, SLV_BOOT.3
- new net N$18: MASTER.(PCI3/MOSI/OC2A)PB3, MST_BOOT.1
- new net N$19: MASTER.(PCI4/MISO)PB4, MST_BOOT.2
- new net N$20: MASTER.(PCI5/SCK)PB5, MST_BOOT.3
- new net N$22: SLAVE.(PCI16/RXD)PD0, SLV_PRGM.2
- new net N$23: SLAVE.(PCI17/TXD)PD1, SLV_PRGM.3
- new net N$24: MASTER.(PCI16/RXD)PD0, MST_PRGM.2
- new net N$25: MASTER.(PCI17/TXD)PD1, MST_PRGM.3
- net +5V: now also BUTTON-2.S, DISPLAY.3, ENC-4.S; no longer SV1.3, X4-4.S, X5-2.S
- net GND: now also DISPLAY.2, ENC-5.S, PWR_IN-1.S; no longer SV1.2, X3-1.S, X4-5.S
- net N$1: now also MST_BOOT.4, MST_PRGM.1
- net N$10: now also ENC-2.S; no longer X4-2.S
- net N$12: now also ENC-1.S; no longer X4-1.S
- net N$14: now also BUTTON-1.S, MASTER.(PCI2/SS/OC1B)PB2; no longer MASTER.(PCI3/MOSI/OC2A)PB3, X5-1.S
- net N$2: now also SLV_BOOT.4, SLV_PRGM.1
- net N$8: now also DISPLAY.1; no longer SV1.1
- net N$9: now also ENC-3.S; no longer X4-3.S
- net VCC: now also PWR_IN-2.S; no longer X3-2.S
Other:
- moved on the sheet: Q2, R3
